Commit message: launch file for simulation added

File: robot_model/description/robot.urdf.xacro (robot description, xacro)
@@ -3,6 +3,6 @@
     <!-- Example link -->
     <xacro:include filename="robot_core.xacro"/>
-    <!-- <xacro:include filename="lidar.xacro" />
-    <xacro:include filename="gazebo_control.xacro" /> -->
+    <!-- <xacro:include filename="lidar.xacro" /> -->
+    <xacro:include filename="gazebo_control.xacro" />
     <!-- <xacro:include filename="ros2_control.xacro" /> -->
 </robot>

File: robot_model/description/robot_core.xacro (robot description, xacro)
@@ -8,5 +8,5 @@
     <xacro:property name="chassis_height" value="0.15"/>
     <xacro:property name="chassis_weight" value="0.5"/>
-    <xacro:include filename="inertial_macro.xacro"/>
+    <xacro:include filename="inertial_macros.xacro"/>
     <material name="white">
         <color rgba="1 1 1 1"/>
@@ -53,5 +53,5 @@
     <!-- LEFT WHEEL LINK-->
     <joint name="left_wheel_joint" type="continuous">
-        <parent link="base_line"/>
+        <parent link="base_link"/>
         <child link="left_wheel"/>
         <origin xyz="0 0.175 0" rpy="-${pi/2} 0 0"/>
@@ -70,4 +70,7 @@
             </geometry>
         </collision>
+        <xacro:inertial_cylinder mass="0.1" length="0.04" radius="0.05">
+            <origin xyz="0 0 0" rpy="0 0 0"/>
+        </xacro:inertial_cylinder>
     </link>
     <gazebo reference="left_wheel">

Commit message: robot model added

File: robot_model/description/robot.urdf.xacro (robot description, xacro)
@@ -3,6 +3,8 @@
     <!-- Example link -->
     <xacro:include filename="robot_core.xacro"/>
-    <!-- <xacro:include filename="lidar.xacro" />
-    <xacro:include filename="gazebo_control.xacro" /> -->
+    <xacro:include filename="lidar.xacro" />
+    <xacro:include filename="imu.xacro"/>
+    <!-- <xacro:include filename="odom.xacro"/> -->
+    <xacro:include filename="gazebo_control.xacro" />
     <!-- <xacro:include filename="ros2_control.xacro" /> -->
 </robot>

File: robot_model/description/robot_core.xacro (robot description, xacro)
@@ -8,5 +8,5 @@
     <xacro:property name="chassis_height" value="0.15"/>
     <xacro:property name="chassis_weight" value="0.5"/>
-    <xacro:include filename="inertial_macro.xacro"/>
+    <xacro:include filename="inertial_macros.xacro"/>
     <material name="white">
         <color rgba="1 1 1 1"/>
@@ -24,4 +24,11 @@
     <link name="base_link">
     </link>
+    <!-- BASE_FOOTPRINT LINK-->
+    <joint name="base_footprint_joint" type="fixed">
+        <parent link="base_link"/>
+        <child link="base_footprint"/>
+        <origin xyz="0 0 0" rpy="0 0 0"/>
+    </joint>
+    <link name="base_footprint"></link>
     <!-- CHASSIS LINK-->
     <joint name="chassis_joint" type="fixed">
@@ -53,5 +60,5 @@
     <!-- LEFT WHEEL LINK-->
     <joint name="left_wheel_joint" type="continuous">
-        <parent link="base_line"/>
+        <parent link="base_link"/>
         <child link="left_wheel"/>
         <origin xyz="0 0.175 0" rpy="-${pi/2} 0 0"/>
@@ -70,4 +77,7 @@
             </geometry>
         </collision>
+        <xacro:inertial_cylinder mass="0.1" length="0.04" radius="0.05">
+            <origin xyz="0 0 0" rpy="0 0 0"/>
+        </xacro:inertial_cylinder>
     </link>
     <gazebo reference="left_wheel">
@@ -128,16 +138,10 @@
     </gazebo>
     <!-- LASER LINK-->
-    <link name="laser"></link>
+    <!-- <link name="laser"></link>
     <joint name="laser_joint" type="fixed">
         <parent link="base_link"/>
         <child link="laser"/>
         <origin xyz="0.1086 0 0.28" rpy="${pi} 0 0"/>
-    </joint>
+    </joint> -->
     <!-- IMU LINK-->
-    <link name="imu_link"></link>
-    <joint name="imu_joint" type="fixed">
-        <parent link="base_link"/>
-        <child link="imu_link"/>
-        <origin xyz="0.075 -0.075 0.1" rpy="${pi} 0 0"/>
-    </joint>
 </robot>
