Commit message: robot autonomous building map added

File: robot_model/description/gazebo_control.xacro (robot description, xacro)
@@ -16,8 +16,8 @@
             <!-- Output -->
             <odometryFrame>odom</odometryFrame>
-            <robotBaseFrame>base_link</robotBaseFrame>
+            <robotBaseFrame>base_footprint</robotBaseFrame>
             <publishOdom>true</publishOdom>
-            <publishOdomTF>true</publishOdomTF>
-            <publishWheelTF>true</publishWheelTF>
+            <publishOdomTF>false</publishOdomTF>
+            <publishWheelTF>false</publishWheelTF>
         </plugin>
     </gazebo>

File: robot_model/description/imu.xacro (robot description, xacro)
@@ -14,8 +14,9 @@
             <robotNamespace>/</robotNamespace>
             <topicName>/imu</topicName>
-            <bodyName>base_link</bodyName>
+            <bodyName>imu_link</bodyName>
+            <frameName>imu_link</frameName>
             <!-- Additional IMU plugin configuration -->
             <!-- <imuTopicName>/imu</imuTopicName> -->
-            <updateRate>50</updateRate>
+            <updateRate>30</updateRate>
         </plugin>
     </gazebo>

File: robot_model/description/odom.xacro (robot description, xacro)
@@ -2,18 +2,6 @@
 <robot xmlns:xacro="http://www.ros.org/wiki/xacro" >
     <!-- Odom LINK -->
-    <joint name="odom_to_base_footprint" type="fixed">
-        <parent link="odom"/>
-        <child link="base_footprint"/>
-        <origin xyz="0 0 0" rpy="0 0 0"/>  <!-- No offset between odom and base_footprint -->
-    </joint>
     <link name="odom">
         <!-- Odometry link typically doesn't have physical properties but is required for EKF -->
     </link>
-    <gazebo>
-        <plugin name="gazebo_ros_odometry" filename="libgazebo_ros_odometry.so">
-            <robotNamespace>/</robotNamespace>
-            <topicName>/odom</topicName>
-            <!-- Additional configuration for the odometry plugin -->
-        </plugin>
-    </gazebo>
 </robot>

File: robot_model/description/robot_core.xacro (robot description, xacro)
@@ -26,6 +26,6 @@
     <!-- BASE_FOOTPRINT LINK-->
     <joint name="base_footprint_joint" type="fixed">
-        <parent link="base_link"/>
-        <child link="base_footprint"/>
+        <parent link="base_footprint"/>
+        <child link="base_link"/>
         <origin xyz="0 0 0" rpy="0 0 0"/>
     </joint>

Commit message: imu and odom xacro added, slamtoolbox launcher added

File: robot_model/description/gazebo_control.xacro (robot description, xacro)
@@ -3,4 +3,10 @@
     <gazebo>
         <plugin name="diff_drive" filename="libgazebo_ros_diff_drive.so">
+            <!-- ROS2 相关配置 -->
+            <ros>
+                <namespace>/</namespace>
+                <remapping>cmd_vel:=cmd_vel</remapping>
+                <remapping>odom:=odom</remapping>
+            </ros>
             <!-- Wheel Information -->
             <left_joint>left_wheel_joint</left_joint>
@@ -13,8 +19,9 @@
             <!-- Output -->
             <odometry_frame>odom</odometry_frame>
-            <robot_base_frame>base_link</robot_base_frame>
+            <robot_base_frame>base_footprint</robot_base_frame>
             <publish_odom>true</publish_odom>
             <publish_odom_tf>true</publish_odom_tf>
-            <publish_wheel_tf>true</publish_wheel_tf>
+            <publish_wheel_tf>false</publish_wheel_tf>
+            <update_rate>50</update_rate>
         </plugin>
     </gazebo>

File: robot_model/description/lidar.xacro (robot description, xacro)
@@ -38,5 +38,5 @@
                 <scan>
                     <horizontal>
-                        <samples>360</samples>
+                        <samples>1440</samples>
                         <min_angle>-3.14</min_angle>
                         <max_angle>3.14</max_angle>

File: robot_model/description/robot.urdf.xacro (robot description, xacro)
@@ -4,4 +4,5 @@
     <xacro:include filename="robot_core.xacro"/>
     <xacro:include filename="lidar.xacro" />
+    <xacro:include filename="imu.xacro"/>
     <xacro:include filename="gazebo_control.xacro" />
     <!-- <xacro:include filename="ros2_control.xacro" /> -->

File: robot_model/description/robot_core.xacro (robot description, xacro)
@@ -26,6 +26,6 @@
     <!-- BASE_FOOTPRINT LINK-->
     <joint name="base_footprint_joint" type="fixed">
-        <parent link="base_link"/>
-        <child link="base_footprint"/>
+        <parent link="base_footprint"/>
+        <child link="base_link"/>
         <origin xyz="0 0 0" rpy="0 0 0"/>
     </joint>
@@ -145,4 +145,5 @@
     </joint> -->
     <!-- IMU LINK-->
+<!--
     <link name="imu_link"></link>
     <joint name="imu_joint" type="fixed">
@@ -150,4 +151,4 @@
         <child link="imu_link"/>
         <origin xyz="0.075 -0.075 0.1" rpy="${pi} 0 0"/>
-    </joint>
+    </joint> -->
 </robot>
